File: controller/controller.kicad_sch (KiCad schematic)
At the start: 30 parts, among them Q1 BSS138, U1 AMS1117-3.3, U2 ESP32-WROOM-E

Commit message: ws2812c library import
Other:
- note added: "User buttons"
- moved on the sheet: C3, C4, C5, C6, R5, R6, R7, R8, R9, SW_1, SW_2, SW_3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
